Commit message: urdf version-2 improved urdf structuring

File: src/roboarm_urdf_description/urdf/roboArm_urdf.urdf.xacro (robot description, xacro)
@@ -14,276 +14,10 @@
         <inertial>
             <mass value="${mass}"/>
-            <inertia    ixx="1.0" ixy="0.0" ixz="0.0"
-                        iyy="1.0" iyz="0.0"
-                        izz="1.0"/>
+            <inertia
+                    ixx="1.0" ixy="0.0" ixz="0.0"
+                    iyy="1.0" iyz="0.0"
+                    izz="1.0"/>
         </inertial>
     </xacro:macro>
-    <!-- For Global coords hence no attributes to it -->
-     <!-- understand it as waist-->
-    <link name="world"/>
-    <!-- base link of the robotarm -->
-    <link name="base_link">
-        <xacro:default_inertial_matrix mass="1.0"/>
-        <!-- within visuals we care about the rendering of the items -->
-        <visual>
-            <!-- origin-tag takes care about orientation(rpy) & position(xyz) w.r.t "base link"-->
-            <!-- <origin rpy="0 0 0" xyz= "-0.45 -0.48 0"/> origin-tag gives pose for the geometry tage elements -->
-            <origin rpy="0 0 0" xyz= "0 0 .175"/> <!-- origin-tag gives pose for the geometry tage elements-->
-            <!-- geometry-tag contains diff object[cylinder, box, sphere..etc] or even meshes that also import ext custom objects -->
-            <geometry>
-                <!-- mesh-tag imports the external part design into the rViz(eg: .STL) -->
-                <!-- <mesh filename="package://roboarm_urdf_description/meshes/basement.STL" scale="0.01 0.01 0.01"/> -->
-                <box size="0.5 0.5 0.34"/>
-            </geometry>
-        </visual>
-        <!-- for Gazebo -->
-        <collision>
-            <!-- <origin rpy="0 0 0" xyz= "-0.45 -0.48 0"/>
-            <geometry>
-                <mesh filename="package://roboarm_urdf_description/meshes/basement.STL" scale="0.01 0.01 0.01"/>
-            </geometry> -->
-            <origin rpy="0 0 0" xyz= "0 0 .175"/>
-            <geometry>
-                <box size="0.5 0.5 0.34"/>
-            </geometry>
-        </collision>
-    </link>
-    <!-- This joint connects the baselink and world so world coords and baselink coord will superimpose -->
-    <!-- the baselink will be fixed and orient as world orient -->
-    <joint name="virtual_joint" type="fixed"> <!-- virtual_joint -->
-        <parent link="world"/>      <!-- previous link-->
-        <child link="base_link"/>   <!-- current link-->
-        <origin rpy="0 0 0" xyz="0 0 0"/> <!--pose of the joint-->
-        <!-- <limit lower="-${PI/2}" upper="${PI/2}" effort="${effort}" velocity="${velocity}"/> -->
-    </joint>
-    <link name="base_plate">   <!-- for tutorials biceps_link = foward_drive_link -->
-        <xacro:default_inertial_matrix mass="0.1"/>
-        <visual>
-            <!-- <origin rpy="0 0 0" xyz="-0.39 -0.39 -0.56"/> -->
-            <origin rpy="0 0 0" xyz="0 0 0.176"/>
-            <geometry>
-                <!-- <mesh filename="package://roboarm_urdf_description/meshes/base_plate.STL" scale="0.01 0.01 0.01"/> -->
-                <box size="0.12 0.12 0.35"/>
-            </geometry>
-        </visual>
-        <!-- for Gazebo -->
-        <collision>
-            <!-- <origin rpy="0 0 0" xyz="-0.39 -0.39 -0.56"/>
-            <geometry>
-                <mesh filename="package://roboarm_urdf_description/meshes/base_plate.STL" scale="0.01 0.01 0.01"/>
-            </geometry> -->
-            <!-- <origin rpy="0 0 0" xyz="-0.39 -0.39 -0.56"/> -->
-            <origin rpy="0 0 0" xyz="0 0 0.176"/>
-            <geometry>
-                <!-- <mesh filename="package://roboarm_urdf_description/meshes/base_plate.STL" scale="0.01 0.01 0.01"/> -->
-                <box size="0.12 0.12 0.35"/>
-            </geometry>
-        </collision>
-    </link>
-    <joint name="joint_1" type="revolute">  <!-- shoulder_joint -->
-        <parent link="base_link"/>
-        <child link="base_plate"/>
-        <axis xyz="0 0 1"/> <!-- rotation of the joint the axis about x-axis -->
-        <!-- <origin rpy="0 0 0" xyz="-0.02 0 0.35"/> -->
-        <origin rpy="0 0 0" xyz="0.0 0.0 0.35"/>
-        <limit lower="-${PI}" upper="${PI}" effort="${effort}" velocity="${velocity}"/>
-    </joint>
-    <link name="biceps_link-l2">   <!-- for tutorials biceps_link = foward_drive_link -->
-        <xacro:default_inertial_matrix mass="0.1"/>
-        <visual>
-            <!-- <origin rpy="0 -${PI/2} ${PI/2}" xyz="0.19 0.06 -0.08"/> -->
-            <origin rpy="0 -${PI/2} ${PI/2}" xyz="0.1 0.0 0.5"/>
-            <geometry>
-                <!-- <mesh filename="package://roboarm_urdf_description/meshes/forward_drive_arm.STL" scale="0.01 0.01 0.01"/> -->
-                <box size="1.0 0.2 0.2"/>
-            </geometry>
-        </visual>
-        <!-- for Gazebo -->
-        <collision>
-            <!-- <origin rpy="0 -${PI/2} ${PI/2}" xyz="0.19 0.06 -0.08"/>
-            <geometry>
-                <mesh filename="package://roboarm_urdf_description/meshes/forward_drive_arm.STL" scale="0.01 0.01 0.01"/>
-            </geometry> -->
-            <origin rpy="0 -${PI/2} ${PI/2}" xyz="0.1 0.0 0.5"/>
-            <geometry>
-                <!-- <mesh filename="package://roboarm_urdf_description/meshes/forward_drive_arm.STL" scale="0.01 0.01 0.01"/> -->
-                <box size="1.0 0.2 0.2"/>
-            </geometry>
-        </collision>
-    </link>
-    <joint name="joint_2" type="revolute">  <!-- shoulder_joint -->
-        <parent link="base_plate"/>
-        <child link="biceps_link-l2"/>
-        <axis xyz="1 0 0"/> <!-- rotation of the joint the axis about x-axis -->
-        <!-- <origin rpy="0 0 0" xyz="-0.02 0 0.35"/> -->
-        <origin rpy="0 0 0" xyz="0.08 0.0 0.20"/>
-        <limit lower="-${PI/2}" upper="${PI/2}" effort="${effort}" velocity="${velocity}"/>
-    </joint>
-    <link name="arm_link-l3">
-        <xacro:default_inertial_matrix mass="0.1"/>
-        <visual>
-            <origin rpy="${PI/2} 0 ${PI/2}" xyz="-0.101 0.5 0" />
-            <geometry>
-                <!-- <mesh filename="package://roboarm_urdf_description/meshes/horizontal_arm.STL" scale="0.01 0.01 0.01"/> -->
-                <box size="1.0 0.2 0.2"/>
-            </geometry>
-        </visual>
-        <!-- for Gazebo -->
-        <collision>
-            <!-- <origin rpy="${PI/2} 0 ${PI/2}" xyz="-0.03 -0.4 -0.06" />
-            <geometry>
-                <mesh filename="package://roboarm_urdf_description/meshes/horizontal_arm.STL" scale="0.01 0.01 0.01"/>
-            </geometry> -->
-            <origin rpy="${PI/2} 0 ${PI/2}" xyz="-0.101 0.5 0" />
-            <geometry>
-                <!-- <mesh filename="package://roboarm_urdf_description/meshes/horizontal_arm.STL" scale="0.01 0.01 0.01"/> -->
-                <box size="1.0 0.2 0.2"/>
-            </geometry>
-        </collision>
-    </link>
-    <joint name="joint_3" type="revolute">
-        <parent link="biceps_link-l2"/>
-        <child link="arm_link-l3"/>
-        <axis xyz="1 0 0"/>
-        <origin rpy="0 0 0" xyz="0 0 0.89"/>
-        <limit lower="-${PI/2}" upper="${PI/2}" effort="${effort}" velocity="${velocity}"/>
-    </joint>
-    <link name="palm_link-l4">
-        <xacro:default_inertial_matrix mass="0.1"/>
-        <visual>
-            <origin rpy="${PI/2} 0 ${PI/2}" xyz="0.101 0.5 0" />
-            <geometry>
-                <!-- <mesh filename="package://roboarm_urdf_description/meshes/horizontal_arm.STL" scale="0.01 0.01 0.01"/> -->
-                <box size="1.0 0.2 0.2"/>
-            </geometry>
-        </visual>
-        <!-- for Gazebo -->
-        <collision>
-            <!-- <origin rpy="${PI/2} 0 ${PI/2}" xyz="-0.03 -0.4 -0.06" />
-            <geometry>
-                <mesh filename="package://roboarm_urdf_description/meshes/horizontal_arm.STL" scale="0.01 0.01 0.01"/>
-            </geometry> -->
-            <origin rpy="${PI/2} 0 ${PI/2}" xyz="0.101 0.5 0" />
-            <geometry>
-                <!-- <mesh filename="package://roboarm_urdf_description/meshes/horizontal_arm.STL" scale="0.01 0.01 0.01"/> -->
-                <box size="1.0 0.2 0.2"/>
-            </geometry>
-        </collision>
-    </link>
-    <!-- for wrist_joint -->
-    <joint name="joint_4" type="revolute">
-        <parent link="arm_link-l3"/>
-        <child link="palm_link-l4"/>
-        <axis xyz="1 0 0"/>
-        <origin rpy="0 0 0" xyz="0 0.6 0"/>
-        <limit lower="-${PI/2}" upper="${PI/2}" effort="${effort}" velocity="${velocity}"/>
-    </joint>
-    <link name="prismatic_link">
-        <xacro:default_inertial_matrix mass="0.05"/>
-        <visual>
-            <origin rpy="${PI/2} 0 ${PI/2}" xyz="-0.11 0.45 0" />
-            <geometry>
-                <!-- <mesh filename="package://roboarm_urdf_description/meshes/horizontal_arm.STL" scale="0.01 0.01 0.01"/> -->
-                <box size="1.0 0.2 0.2"/>
-            </geometry>
-        </visual>
-        <!-- for Gazebo -->
-        <collision>
-            <!-- <origin rpy="0 0 ${PI/2}" xyz="0 -0.05 -0.15"/> -->
-            <origin rpy="0 0 ${PI/2}" xyz="-0.11 0.45 0" />
-            <geometry>
-                <!-- <mesh filename="package://roboarm_urdf_description/meshes/claw_support.STL" scale="0.01 0.01 0.01"/> -->
-                <box size="1.0 0.2 0.2"/>
-            </geometry>
-        </collision>
-    </link>
-    <joint name="joint_prism" type="prismatic">
-        <parent link="palm_link-l4"/>
-        <child link="prismatic_link"/>
-        <axis xyz="0 1 0"/>
-        <origin rpy="0 0 0" xyz="0 0.5 0"/>
-        <limit lower="0.0" upper="0.50"
-           effort="10.0" velocity="0.05"/>
-    </joint>
-    <!-- for tutorial palm = claw_support-->
-    <link name="claw_link-l5">
-        <xacro:default_inertial_matrix mass="0.05"/>
-        <visual>
-            <!-- <origin rpy="0 0 ${PI/2}" xyz="0 -0.05 -0.15"/> -->
-            <origin rpy="0 0 ${PI/2}" xyz="0 0.0 0.0" />
-            <geometry>
-                <!-- <mesh filename="package://roboarm_urdf_description/meshes/claw_support.STL" scale="0.01 0.01 0.01"/> -->
-                <box size="0.12 0.25 0.25"/>
-            </geometry>
-        </visual>
-        <!-- for Gazebo -->
-        <collision>
-            <!-- <origin rpy="0 0 ${PI/2}" xyz="0 -0.05 -0.15"/> -->
-            <origin rpy="0 0 ${PI/2}" xyz="0 0.0 0.0" />
-            <geometry>
-                <!-- <mesh filename="package://roboarm_urdf_description/meshes/claw_support.STL" scale="0.01 0.01 0.01"/> -->
-                <box size="0.12 0.25 0.25"/>
-            </geometry>
-        </collision>
-    </link>
-    <!-- nuckles_joint -->
-    <joint name="nuckles_joint" type="fixed">
-        <parent link="prismatic_link"/>
-        <child link="claw_link-l5"/>
-        <origin rpy="0 0 0" xyz="-0.125 1.01 0"/>
-    </joint>
-    <!-- finger-->
-    <link name="gripper_right">
-        <xacro:default_inertial_matrix mass="0.01"/>
-        <visual>
-            <origin rpy="0 0 -${PI/2}" xyz="-0.1 0.6 0.0"/>
-            <geometry>
-                <mesh filename="package://roboarm_urdf_description/meshes/right_finger.STL" scale="0.01 0.01 0.01"/>
-            </geometry>
-        </visual>
-        <!-- for Gazebo -->
-        <collision>
-            <origin rpy="0 0 -${PI/2}" xyz="-0.1 0.6 0.0"/>
-            <geometry>
-                <mesh filename="package://roboarm_urdf_description/meshes/right_finger.STL" scale="0.01 0.01 0.01"/>
-            </geometry>
-        </collision>
-    </link>
-    <!--finger-->
-    <link name="gripper_left">
-        <xacro:default_inertial_matrix mass="0.01"/>
-        <visual>
-            <!-- <origin rpy="0 0 -${PI/2}" xyz="-0.04 0.5 -0.1"/> -->
-            <origin rpy="0 0 -${PI/2}" xyz="-0.04 0.6 0.0"/>
-            <geometry>
-                <mesh filename="package://roboarm_urdf_description/meshes/left_finger.STL" scale="0.01 0.01 0.01"/>
-            </geometry>
-        </visual>
-        <!-- for Gazebo -->
-        <collision>
-           <origin rpy="0 0 -${PI/2}" xyz="-0.04 0.6 0.0"/>
-            <geometry>
-                <mesh filename="package://roboarm_urdf_description/meshes/left_finger.STL" scale="0.01 0.01 0.01"/>
-            </geometry>
-        </collision>
-    </link>
-    <!-- for gripperRight_joint -->
-    <joint name="joint_5" type="revolute">
-        <parent link="claw_link-l5"/>
-        <child link="gripper_right"/>
-        <axis xyz="0 0 1"/>
-        <!-- <origin rpy="0 0 0" xyz="-0.04 0.13 -0.1"/> -->
-        <origin rpy="0 0 0" xyz="+0.07 0.13 0.0"/>
-        <limit lower="-${PI/2}" upper="0.0" effort="${effort}" velocity="${velocity}"/>
-    </joint>
-    <!-- for gripperLeft_joint -->
-    <joint name="joint_6" type="revolute">
-        <parent link="claw_link-l5"/>
-        <child link="gripper_left"/>
-        <axis xyz="0 0 1"/>
-        <!-- <origin rpy="0 0 0" xyz="-0.22 0.13 -0.1"/> -->
-        <origin rpy="0 0 0" xyz="-0.09 0.13 0.0"/>
-        <mimic joint="joint_5" multiplier="-1"/>  <!-- it mimics the right_gripper but in apposite way due to multiplier -1-->
-        <limit lower="0" upper="${PI/2}" effort="${effort}" velocity="${velocity}"/>
-    </joint>
+    <xacro:include filename="$(find roboarm_urdf_description)/urdf/roboArm_urdf_descript.urdf.xacro"/>
 </robot>
