Commit message: Added corrected optical camera frame for ROS2 & Added controller for gripper control

File: src/roboarm_urdf_description/urdf/roboArm_ros2_control.urdf.xacro (robot description, xacro)
@@ -35,4 +35,15 @@
             <state_interface name="effort"/>
         </joint>
+        <joint name="joint_5">
+            <command_interface name="position"/>
+            <state_interface name="position"/>
+            <state_interface name="velocity"/>
+            <state_interface name="effort"/>
+        </joint>
+        <joint name="joint_6">
+            <state_interface name="position"/>
+            <state_interface name="velocity"/>
+            <state_interface name="effort"/>
+        </joint>
     </ros2_control>
     <gazebo>

File: src/roboarm_urdf_description/urdf/roboArm_urdf.urdf.xacro (robot description, xacro)
@@ -28,4 +28,5 @@
                 params="mass sx sy sz xyz rpy">
         <inertial>
+            <!-- giving the inertia frame the geometrical position & orientation becuase its important for the inertia frame to align with object's frame location & rotation -->
             <origin xyz="${xyz}" rpy="${rpy}"/>
             <mass value="${mass}"/>

File: src/roboarm_urdf_description/urdf/sensors_description.urdf.xacro (robot description, xacro)
@@ -29,4 +29,11 @@
         <child link="camera_link"/>
     </joint>
+    <!-- Gazebo frame correction for ROS2 -->
+    <link name="corrected_optical_frame"></link>
+    <joint name="optical_joint" type="fixed">
+        <parent link="camera_link"/>
+        <child link="corrected_optical_frame"/>
+        <origin xyz="0 0 0" rpy="${-PI/2} 0 ${-PI/2}"/>
+    </joint>
     <!-- camera gazebo plugin-->
     <gazebo reference="camera_link">
@@ -34,5 +41,7 @@
             <update_rate>30.0</update_rate>
             <topic>/rgbd_camera</topic>
+            <gz_frame_id>camera_link</gz_frame_id>
             <camera>
+                <optical_frame_id>corrected_optical_frame</optical_frame_id>
                 <horizontal_fov>1.3962634</horizontal_fov>
                 <image>
@@ -43,5 +52,5 @@
                 <clip>
                     <near>0.02</near>
-                    <far>300</far>
+                    <far>500</far>
                 </clip>
                 <noise>
