Commit message: added rgbd_camera sensor

File: src/roboarm_urdf_description/urdf/roboArm_description.urdf.xacro (robot description, xacro)
@@ -156,5 +156,5 @@
         <parent link="prismatic_link"/>
         <child link="claw_link"/>
-        <origin rpy="0 0 0" xyz="-0.125 1.01 0"/>
+        <origin rpy="0 0 0" xyz="-0.124 1.01 0"/>
     </joint>
     <!-- finger-->

File: src/roboarm_urdf_description/urdf/roboArm_urdf.urdf.xacro (robot description, xacro)
@@ -2,12 +2,14 @@
 <robot xmlns:xacro="http://www.ros.org/wiki/xacro" name="Robot_Arm" >
     <xacro:arg name="use_gazebo" default="true"/>
-    <xacro:if value="$(arg use_gazebo)">
+    <!-- <xacro:if value="$(arg use_gazebo)">
         <xacro:include filename="$(find roboarm_urdf_description)/urdf/roboArm_gazebo.xacro"/>
         <xacro:include filename="$(find roboarm_urdf_description)/urdf/roboArm_ros2_control.xacro"/>
-    </xacro:if>
+    </xacro:if>     -->
     <!-- xacro:property is also variable - but for local use not like xacro:arg -->
     <xacro:property name="PI" value="3.141592653589793"/>
     <xacro:property name="effort" value="3.0"/>
     <xacro:property name="velocity" value="5.0"/>
+    <!-- Size of square 'camera' box -->
+    <xacro:property name="camera_link" value="0.1" />
     <!-- inertial matrix for Gazebo simulation for each link hence here as global varibale -->
     <xacro:macro name="default_inertial_matrix" params="mass">
@@ -20,4 +22,5 @@
         </inertial>
     </xacro:macro>
-    <xacro:include filename="$(find roboarm_urdf_description)/urdf/roboArm_urdf_descript.urdf.xacro"/>
+    <xacro:include filename="$(find roboarm_urdf_description)/urdf/roboArm_description.urdf.xacro"/>
+    <xacro:include filename="$(find roboarm_urdf_description)/urdf/sensors_description.urdf.xacro"/>
 </robot>

Commit message: add world elements & resolved unstable motion & temporary camera view fixing

File: src/roboarm_urdf_description/urdf/roboArm_description.urdf.xacro (robot description, xacro)
@@ -3,5 +3,7 @@
     <!-- base link of the robotarm -->
     <link name="base_link">
-        <xacro:default_inertial_matrix mass="1.0"/>
+        <xacro:box_inertial
+            mass="1.0" sx="0.5" sy="0.5" sz="0.34"
+            xyz="0 0 0.175" rpy="0 0 0"/>
         <visual>
            <origin rpy="0 0 0" xyz= "0 0 .175"/>
@@ -24,5 +26,7 @@
     </joint>
     <link name="base_plate">
-        <xacro:default_inertial_matrix mass="0.1"/>
+        <xacro:box_inertial
+            mass="1.0" sx="0.12" sy="0.12" sz="0.35"
+            xyz="0 0 0.176" rpy="0 0 0"/>
         <visual>
             <origin rpy="0 0 0" xyz="0 0 0.176"/>
@@ -43,8 +47,10 @@
         <axis xyz="0 0 1"/>
         <origin rpy="0 0 0" xyz="0.0 0.0 0.35"/>
-        <limit lower="-${PI}" upper="${PI}" effort="${effort}" velocity="${velocity}"/>
+        <limit lower="-${PI}" upper="${PI}" effort="${joint_1_effort}" velocity="${velocity}"/>
     </joint>
     <link name="biceps_link">
-        <xacro:default_inertial_matrix mass="0.1"/>
+        <xacro:box_inertial
+            mass="1.0" sx="1.0" sy="0.2" sz="0.2"
+            xyz="0.1 0 0.5" rpy="0 -${PI/2} ${PI/2}"/>
         <visual>
             <origin rpy="0 -${PI/2} ${PI/2}" xyz="0.1 0.0 0.5"/>
@@ -65,8 +71,10 @@
         <axis xyz="1 0 0"/>
         <origin rpy="0 0 0" xyz="0.08 0.0 0.20"/>
-        <limit lower="-${PI/2}" upper="${PI/2}" effort="${effort}" velocity="${velocity}"/>
+        <limit lower="-${PI/2}" upper="${PI/2}" effort="${joint_2_effort}" velocity="${velocity}"/>
     </joint>
     <link name="arm_link">
-        <xacro:default_inertial_matrix mass="0.1"/>
+        <xacro:box_inertial
+            mass="1.0" sx="1.0" sy="0.2" sz="0.2"
+            xyz="-0.101 0.5 0" rpy="${PI/2} 0 ${PI/2}"/>
         <visual>
             <origin rpy="${PI/2} 0 ${PI/2}" xyz="-0.101 0.5 0" />
@@ -87,8 +95,10 @@
         <axis xyz="1 0 0"/>
         <origin rpy="0 0 0" xyz="0 0 0.89"/>
-        <limit lower="-${PI/2}" upper="${PI/2}" effort="${effort}" velocity="${velocity}"/>
+        <limit lower="-${PI/2}" upper="${PI/2}" effort="${joint_3_effort}" velocity="${velocity}"/>
     </joint>
     <link name="wrist_link">
-        <xacro:default_inertial_matrix mass="0.1"/>
+        <xacro:box_inertial
+            mass="1.0" sx="1.0" sy="0.2" sz="0.2"
+            xyz="0.101 0.5 0" rpy="${PI/2} 0 ${PI/2}"/>
         <visual>
             <origin rpy="${PI/2} 0 ${PI/2}" xyz="0.101 0.5 0" />
@@ -109,8 +119,10 @@
         <axis xyz="1 0 0"/>
         <origin rpy="0 0 0" xyz="0 0.6 0"/>
-        <limit lower="-${PI/2}" upper="${PI/2}" effort="${effort}" velocity="${velocity}"/>
+        <limit lower="-${PI/2}" upper="${PI/2}" effort="${joint_4_effort}" velocity="${velocity}"/>
     </joint>
     <link name="prismatic_link">
-        <xacro:default_inertial_matrix mass="0.05"/>
+        <xacro:box_inertial
+            mass="1.0" sx="1.0" sy="0.2" sz="0.2"
+            xyz="-0.11 0.45 0" rpy="${PI/2} 0 ${PI/2}"/>
         <visual>
             <origin rpy="${PI/2} 0 ${PI/2}" xyz="-0.11 0.45 0" />
@@ -133,8 +145,10 @@
         <origin rpy="0 0 0" xyz="0 0.5 0"/>
         <limit lower="0.0" upper="0.50"
-           effort="10.0" velocity="0.05"/>
+           effort="${joint_prism_effort}" velocity="0.05"/>
     </joint>
     <link name="claw_link">
-        <xacro:default_inertial_matrix mass="0.05"/>
+        <xacro:box_inertial
+            mass="0.5" sx="0.12" sy="0.25" sz="0.25"
+            xyz="0 0 0" rpy="0 0 ${PI/2}"/>
         <visual>
             <origin rpy="0 0 ${PI/2}" xyz="0 0.0 0.0" />
@@ -160,5 +174,5 @@
     <!-- finger-->
     <link name="gripper_right">
-        <xacro:default_inertial_matrix mass="0.01"/>
+        <xacro:default_inertial_matrix mass="0.1"/>
         <visual>
             <origin rpy="0 0 -${PI/2}" xyz="-0.1 0.6 0.0"/>
@@ -177,5 +191,5 @@
     <!--finger-->
     <link name="gripper_left">
-        <xacro:default_inertial_matrix mass="0.01"/>
+        <xacro:default_inertial_matrix mass="0.1"/>
         <visual>
             <origin rpy="0 0 -${PI/2}" xyz="-0.04 0.6 0.0"/>
@@ -198,5 +212,5 @@
         <axis xyz="0 0 1"/>
         <origin rpy="0 0 0" xyz="+0.07 0.13 0.0"/>
-        <limit lower="-${PI/2}" upper="0.0" effort="${effort}" velocity="${velocity}"/>
+        <limit lower="-${PI/2}" upper="0.0" effort="${joint_prism_effort}" velocity="${velocity}"/>
     </joint>
     <!-- for gripperLeft_joint -->
@@ -207,5 +221,5 @@
         <origin rpy="0 0 0" xyz="-0.09 0.13 0.0"/>
         <mimic joint="joint_5" multiplier="-1"/>  <!-- it mimics the right_gripper but in apposite way due to multiplier -1-->
-        <limit lower="0" upper="${PI/2}" effort="${effort}" velocity="${velocity}"/>
+        <limit lower="0" upper="${PI/2}" effort="${joint_prism_effort}" velocity="${velocity}"/>
     </joint>
 </robot>

File: src/roboarm_urdf_description/urdf/roboArm_urdf.urdf.xacro (robot description, xacro)
@@ -7,5 +7,9 @@
     <!-- xacro:property is also variable - but for local use not like xacro:arg -->
     <xacro:property name="PI" value="3.141592653589793"/>
-    <xacro:property name="effort" value="3.0"/>
+    <xacro:property name="joint_1_effort" value="20.0"/>
+    <xacro:property name="joint_2_effort" value="120.0"/>
+    <xacro:property name="joint_3_effort" value="120.0"/>
+    <xacro:property name="joint_4_effort" value="70.0"/>
+    <xacro:property name="joint_prism_effort" value="50.0"/>
     <xacro:property name="velocity" value="5.0"/>
     <!-- Size of square 'camera' box -->
@@ -16,7 +20,21 @@
             <mass value="${mass}"/>
             <inertia
-                    ixx="1.0" ixy="0.0" ixz="0.0"
+                    ixx="1.0" ixy="0.0" ixz="0.00"
                     iyy="1.0" iyz="0.0"
                     izz="1.0"/>
+        </inertial>
+    </xacro:macro>
+    <xacro:macro name="box_inertial"
+                params="mass sx sy sz xyz rpy">
+        <inertial>
+            <origin xyz="${xyz}" rpy="${rpy}"/>
+            <mass value="${mass}"/>
+            <inertia
+                ixx="${mass * (sy*sy + sz*sz) / 12.0}"
+                ixy="0.0"
+                ixz="0.0"
+                iyy="${mass * (sx*sx + sz*sz) / 12.0}"
+                iyz="0.0"
+                izz="${mass * (sx*sx + sy*sy) / 12.0}"/>
         </inertial>
     </xacro:macro>

File: src/roboarm_urdf_description/urdf/sensors_description.urdf.xacro (robot description, xacro)
@@ -24,5 +24,6 @@
     <joint name="camera_joint" type="fixed">
         <axis xyz="0 1 0" />
-        <origin xyz="0 0 0.175" rpy="0 0 0"/>
+        <!-- Orientation of the camera view is controlled by rpy in the origin tag -->
+        <origin xyz="0 0 0.175" rpy="0 0 ${PI/2}"/>
         <parent link="claw_link"/>
         <child link="camera_link"/>

Commit message: made perception package and Implemented HSV based detection and 2D image detection

File: src/roboarm_urdf_description/urdf/roboArm_description.urdf.xacro (robot description, xacro)
@@ -119,5 +119,5 @@
         <axis xyz="1 0 0"/>
         <origin rpy="0 0 0" xyz="0 0.6 0"/>
-        <limit lower="-${PI/2}" upper="${PI/2}" effort="${joint_4_effort}" velocity="${velocity}"/>
+        <limit lower="-${PI}" upper="${PI}" effort="${joint_4_effort}" velocity="${velocity}"/>
     </joint>
     <link name="prismatic_link">
