Commit message: toboarm_moveit2 version updated due to update in URDF version

File: src/roboarm_movit_config/config/Robot_Arm.ros2_control.xacro (robot description, xacro)
@@ -10,50 +10,31 @@
             <joint name="joint_1">
                 <command_interface name="position"/>
-                <!-- <command_interface name="velocity"/>
-                <command_interface name="effort"/> -->
-                <state_interface name="position">
-                  <param name="initial_value">${initial_positions['joint_1']}</param>
-                </state_interface>
                 <state_interface name="velocity"/>
-                <state_interface name="effort"/>
+                <state_interface name="position"/>
             </joint>
             <joint name="joint_2">
                 <command_interface name="position"/>
-                <!-- <command_interface name="velocity"/>
-                <command_interface name="effort"/> -->
-                <state_interface name="position">
-                  <param name="initial_value">${initial_positions['joint_2']}</param>
-                </state_interface>
                 <state_interface name="velocity"/>
-                <state_interface name="effort"/>
+                <state_interface name="position"/>
             </joint>
             <joint name="joint_3">
                 <command_interface name="position"/>
-                <!-- <command_interface name="velocity"/>
-                <command_interface name="effort"/> -->
-                <state_interface name="position">
-                  <param name="initial_value">${initial_positions['joint_3']}</param>
-                </state_interface>
                 <state_interface name="velocity"/>
-                <state_interface name="effort"/>
+                <state_interface name="position"/>
             </joint>
             <joint name="joint_4">
                 <command_interface name="position"/>
-                <!-- <command_interface name="velocity"/>
-                <command_interface name="effort"/> -->
-                <state_interface name="position">
-                  <param name="initial_value">${initial_positions['joint_4']}</param>
-                </state_interface>
                 <state_interface name="velocity"/>
-                <state_interface name="effort"/>
+                <state_interface name="position"/>
+            </joint>
+            <joint name="joint_prism">
+                <command_interface name="position"/>
+                <state_interface name="velocity"/>
+                <state_interface name="position"/>
             </joint>
             <joint name="joint_5">
                 <command_interface name="position"/>
-                <!-- <command_interface name="velocity"/>
-                <command_interface name="effort"/> -->
-                <state_interface name="position">
-                  <param name="initial_value">${initial_positions['joint_5']}</param>
-                </state_interface>
                 <state_interface name="velocity"/>
+                <state_interface name="position"/>
                 <state_interface name="effort"/>
             </joint>

File: src/roboarm_urdf_description/urdf/roboArm_urdf_descript.urdf.xacro (robot description, xacro)
@@ -38,5 +38,5 @@
         </collision>
     </link>
-    <joint name="joint-1" type="revolute">
+    <joint name="joint_1" type="revolute">
         <parent link="base_link"/>
         <child link="base_plate"/>

Commit message: Add depth detection and received the X,Y,Z coodinates of the object in realworld

File: src/roboarm_movit_config/config/Robot_Arm.ros2_control.xacro (robot description, xacro)
@@ -10,31 +10,55 @@
             <joint name="joint_1">
                 <command_interface name="position"/>
+                <state_interface name="position">
+                  <param name="initial_value">${initial_positions['joint_1']}</param>
+                </state_interface>
                 <state_interface name="velocity"/>
-                <state_interface name="position"/>
+                <state_interface name="effort"/>
             </joint>
             <joint name="joint_2">
                 <command_interface name="position"/>
+                <state_interface name="position">
+                  <param name="initial_value">${initial_positions['joint_2']}</param>
+                </state_interface>
                 <state_interface name="velocity"/>
-                <state_interface name="position"/>
+                <state_interface name="effort"/>
             </joint>
             <joint name="joint_3">
                 <command_interface name="position"/>
+                <state_interface name="position">
+                  <param name="initial_value">${initial_positions['joint_3']}</param>
+                </state_interface>
                 <state_interface name="velocity"/>
-                <state_interface name="position"/>
+                <state_interface name="effort"/>
             </joint>
             <joint name="joint_4">
                 <command_interface name="position"/>
+                <state_interface name="position">
+                  <param name="initial_value">${initial_positions['joint_4']}</param>
+                </state_interface>
                 <state_interface name="velocity"/>
-                <state_interface name="position"/>
+                <state_interface name="effort"/>
             </joint>
             <joint name="joint_prism">
                 <command_interface name="position"/>
+                <state_interface name="position">
+                  <param name="initial_value">${initial_positions['joint_prism']}</param>
+                </state_interface>
                 <state_interface name="velocity"/>
-                <state_interface name="position"/>
+                <state_interface name="effort"/>
             </joint>
             <joint name="joint_5">
                 <command_interface name="position"/>
+                <state_interface name="position">
+                  <param name="initial_value">${initial_positions['joint_5']}</param>
+                </state_interface>
                 <state_interface name="velocity"/>
-                <state_interface name="position"/>
+                <state_interface name="effort"/>
+            </joint>
+            <joint name="joint_6">
+                <state_interface name="position">
+                    <param name="initial_value">${initial_positions['joint_6']}</param>
+                </state_interface>
+                <state_interface name="velocity"/>
                 <state_interface name="effort"/>
             </joint>

File: src/roboarm_movit_config/config/Robot_Arm.urdf.xacro (robot description, xacro)
@@ -2,5 +2,4 @@
 <robot xmlns:xacro="http://www.ros.org/wiki/xacro" name="Robot_Arm">
     <xacro:arg name="initial_positions_file" default="initial_positions.yaml" />
-    <xacro:arg name="use_gazebo" default="false"/>
     <!-- Import Robot_Arm urdf file -->
     <xacro:include filename="$(find roboarm_urdf_description)/urdf/roboArm_urdf.urdf.xacro" />

Commit message: Added - Depth images converted to point cloud 3D coordinates are also generated + performing roboarm motion to the target loction using movit2

File: src/roboarm_movit_config/config/Robot_Arm.ros2_control.xacro (robot description, xacro)
@@ -14,5 +14,4 @@
                 </state_interface>
                 <state_interface name="velocity"/>
-                <state_interface name="effort"/>
             </joint>
             <joint name="joint_2">
@@ -22,5 +21,4 @@
                 </state_interface>
                 <state_interface name="velocity"/>
-                <state_interface name="effort"/>
             </joint>
             <joint name="joint_3">
@@ -30,5 +28,4 @@
                 </state_interface>
                 <state_interface name="velocity"/>
-                <state_interface name="effort"/>
             </joint>
             <joint name="joint_4">
@@ -38,5 +35,4 @@
                 </state_interface>
                 <state_interface name="velocity"/>
-                <state_interface name="effort"/>
             </joint>
             <joint name="joint_prism">
@@ -46,5 +42,4 @@
                 </state_interface>
                 <state_interface name="velocity"/>
-                <state_interface name="effort"/>
             </joint>
             <joint name="joint_5">
@@ -54,12 +49,4 @@
                 </state_interface>
                 <state_interface name="velocity"/>
-                <state_interface name="effort"/>
-            </joint>
-            <joint name="joint_6">
-                <state_interface name="position">
-                    <param name="initial_value">${initial_positions['joint_6']}</param>
-                </state_interface>
-                <state_interface name="velocity"/>
-                <state_interface name="effort"/>
             </joint>
         </ros2_control>
